Commit message: refactoring and polishing

File: src/arm_description/urdf/arm.gazebo.xacro (robot description, xacro)
@@ -2,5 +2,5 @@
 <robot xmlns:xacro="http://www.ros.org/wiki/xacro">
   <xacro:macro name="gazebo_tags">
-<!--    gazebo_ros_control plugin-->
+    <!--    gazebo_ros_control plugin-->
     <gazebo>
       <plugin name="gazebo_ros_control" filename="libgazebo_ros_control.so">

File: src/arm_description/urdf/arm.urdf.xacro (robot description, xacro)
@@ -37,6 +37,5 @@
     <collision>
       <geometry>
-<!--        TODO -->
-          <box size="0.05 0.08 0.1"/>
+          <box size="0.07 0.08 0.01"/>
       </geometry>
       <origin rpy="0 0 0" xyz="0 0.012 0.001"/>
@@ -85,9 +84,8 @@
     </visual>
     <collision>
-      <geometry>
-<!--        TODO -->
-           <box size="0.08 0.035 0.045"/>
-        </geometry>
-      <origin rpy="0 0 0" xyz="0 0 0"/>
+      <origin xyz="0.014 0 0" rpy="0 0 0"/> <!-- Adjust position and orientation as needed -->
+      <geometry>
+        <box size="0.058 0.035 0.041"/>
+      </geometry>
     </collision>
      <inertial>
@@ -124,8 +122,8 @@
       <geometry>
           <box size="0.06 0.1 0.035"/>
-        </geometry>
+      </geometry>
       <origin rpy="0 0 0" xyz="0 -0.015 0"/>
     </collision>
-     <inertial>
+    <inertial>
       <mass value="0.1"/>
       <inertia ixx="6.90013881e+01" ixy="0.0" ixz="0.0" iyy="1.24554875e+02" iyz="0.0" izz="1.04295793e+02"/>
@@ -145,9 +143,8 @@
     </visual>
    <collision>
-      <geometry>
-<!--        TODO -->
-          <box size="0.08 0.035 0.045"/>
-        </geometry>
-      <origin rpy="0 0 0" xyz="0 0 0"/>
+       <origin xyz="0.014 0 0" rpy="0 0 0"/> <!-- Adjust position and orientation as needed -->
+       <geometry>
+         <box size="0.058 0.035 0.041"/>
+       </geometry>
     </collision>
      <inertial>
@@ -205,9 +202,8 @@
     </visual>
     <collision>
-      <geometry>
-<!--         TODO -->
-          <box size="0.08 0.035 0.045"/>
-        </geometry>
-      <origin rpy="0 0 0" xyz="0 0 0"/>
+      <origin xyz="0.014 0 0" rpy="0 0 0"/>
+      <geometry>
+        <box size="0.058 0.035 0.041"/>
+      </geometry>
     </collision>
     <inertial>
@@ -265,9 +261,8 @@
     </visual>
     <collision>
-      <geometry>
-<!--        TODO -->
-          <box size="0.08 0.035 0.045"/>
-        </geometry>
-      <origin rpy="0 0 0" xyz="0 0 0"/>
+      <origin xyz="0.014 0 0" rpy="0 0 0"/> <!-- Adjust position and orientation as needed -->
+      <geometry>
+        <box size="0.058 0.035 0.041"/>
+      </geometry>
     </collision>
     <inertial>

File: src/arm_description/urdf/camera.urdf.xacro (robot description, xacro)
@@ -4,5 +4,5 @@
     <xacro:macro name="camera_sensor" params="xyz rpy parent robot_name">
         <joint name="camera_sensor_joint" type="fixed">
-<!--            looking in the forward direction-->
+            <!-- looking in the forward direction-->
             <axis xyz="0 0 1" />
             <origin xyz="${xyz}" rpy="${rpy}"/>
@@ -64,5 +64,5 @@
                 </plugin>
             </sensor>
-<!--            Adding color so that it shows up in Gazebo-->
+            <!-- Adding color for Gazebo-->
             <material>Gazebo/Green</material>
     </gazebo>
